File: Type.1/dummy_keyboard.kicad_pcb (KiCad board)
At the start: 2 copper layers, 50 x 25 mm, 3 parts, among them SW1 SW_Push

Commit message: update: update product type
Parts:
- moved G*** 0.50 mm to (167.0, 103.5)
Other:
- board text added: "Tel. 031-329-4300"
- board text added: "덕영고등학교"
- board text added: "덕영고등학교 메이크동아리"
- board text added: "인공지능SW과, 정보보안SW과, 경영회계과, 빅데이터과, 보건간호과, 그래픽SW과"
- board text removed: "덕영고등학교 소프트웨어부"
