File: Type.3/dummy_keyboard.kicad_pcb (KiCad board)
At the start: 2 copper layers, 50 x 25 mm, 3 parts, among them SW1 SW_Push

Commit message: update: update product type
Parts:
- moved G*** 0.47 mm to (166.1, 102.5)
